Commit message: adding new urdf models and spawing them in the environment

File: assets/urdf/Aurmar_description/objects/cylinder.urdf (robot description, URDF)
Before this commit: robot object_cylinder, 1 links, 0 joints
Links:
- link cylinder: geometry collision cylinder length=0.07 radius=0.035; visual cylinder length=0.07 radius=0.035
