Commit message: added new camera module, added new files to cacluate suction score and changed the urdf file for suction gripper

File: assets/urdf/Aurmar_description/robots/robot_storm.urdf (robot description, URDF)
Before this commit: robot ur, 18 links, 17 joints
Links:
- removed link left_bar
- removed link left_distal_phalanx
- removed link left_outer_knuckle
- removed link left_proximal_phalanx
- removed link right_bar
- removed link right_distal_phalanx
- removed link right_outer_knuckle
- removed link right_proximal_phalanx
- added link epick_end_effector, mass 0.0001; visual cylinder length=0.01 radius=0.0225
- added link epick_rod, mass 0.0001; visual cylinder length=0.1 radius=0.01
- link gripper_link: mass 0.7 -> 0.745; geometry collision cylinder length=0.13 radius=0.044; visual cylinder length=0.03 radius=0.006
Joints:
- removed joint left_bar_joint
- removed joint left_distal_phalanx_joint
- removed joint left_outer_knuckle_joint
- removed joint left_proximal_phalanx_joint
- removed joint right_bar_joint
- removed joint right_distal_phalanx_joint
- removed joint right_outer_knuckle_joint
- removed joint right_proximal_phalanx_joint
- added joint eef_hand_joint: type fixed, parent epick_rod, child epick_end_effector, origin xyz=0 0 0.055 rpy=0 0 0
- added joint rod_joint: type fixed, parent gripper_link, child epick_rod, origin xyz=0 0 0.13 rpy=0 0 0
- joint ee_fixed_joint: origin xyz=0.0 0. 0.1 rpy=0.0 0.0 -1.57 -> xyz=0.0 0.0 0.0 rpy=0.0 0.0 -1.57; parent gripper_link -> epick_end_effector

Commit message: adding  changes for orientation control

File: assets/urdf/Aurmar_description/robots/robot_storm.urdf (robot description, URDF)
Before this commit: robot ur, 12 links, 11 joints
Links:
- link epick_end_effector: geometry collision cylinder length=0.01 radius=0.015; visual cylinder length=0.01 radius=0.0225
- link epick_rod: geometry collision cylinder length=0.1 radius=0.01; visual cylinder length=0.1 radius=0.01
Joints:
- joint ee_fixed_joint: origin xyz=0.0 0.0 0.0 rpy=0.0 0.0 -1.57 -> xyz=0.0 0.0 0.0 rpy=0.0 0.0 0.0

Commit message: adding changes to urdf

File: assets/urdf/Aurmar_description/robots/robot_storm.urdf (robot description, URDF)
Before this commit: robot ur, 12 links, 11 joints
Joints:
- joint gripper_joint: origin xyz=0 0 0 rpy=0 0 90 -> xyz=0 0 0 rpy=0 0 4.7124

Commit message: Adding trasnform file for tensor and making changes in urdf for back plane

File: assets/urdf/Aurmar_description/robots/robot_storm.urdf (robot description, URDF)
Before this commit: robot ur, 12 links, 11 joints
Joints:
- joint ee_fixed_joint: origin xyz=0.0 0.0 0.0 rpy=0.0 0.0 0.0 -> xyz=0.0 0.0 0.0 rpy=0 -1.57 -3.14

Commit message: Adding suction projections and pose sampling

File: assets/urdf/Aurmar_description/robots/robot_storm.urdf (robot description, URDF)
Before this commit: robot ur, 12 links, 11 joints
Links:
- link epick_end_effector: geometry collision cylinder length=0.01 radius=0.02; visual cylinder length=0.01 radius=0.02
Joints:
- joint ee_fixed_joint: origin xyz=0.0 0.0 0.0 rpy=0 -1.57 -3.14 -> xyz=0.0 0.0 -0.005 rpy=0 -1.57 -3.14

Commit message: partial code completion  for parallelization

File: assets/urdf/Aurmar_description/robots/robot_storm.urdf (robot description, URDF)
Before this commit: robot ur, 12 links, 11 joints
Links:
- link ee_link: geometry 
- link epick_end_effector: mass 0.0001 -> 0.01
- link epick_rod: mass 0.0001 -> 0.070; geometry collision cylinder length=0.078 radius=0.0065; visual cylinder length=0.078 radius=0.0065
- link gripper_link: mass 0.745 -> 0.7; geometry collision cylinder length=0.10 radius=0.0385; visual mesh filename=robotiq_epick_visualization/meshes/visual/robotiq_epick.dae scale=0.001 0.001 0.001
Joints:
- joint eef_hand_joint: axis (none) -> 0 0 1; limit (none) -> lower=0.0 upper=0.008 effort=1000.0 velocity=100; origin xyz=0 0 0.055 rpy=0 0 0 -> xyz=0 0 0.053 rpy=0 0 0; type fixed -> prismatic
- joint gripper_joint: limit lower=0 upper=0.8 effort=1000 velocity=0.5 -> (none)
