Commit message: Changes done for google scanned objects integration

File: assets/urdf/Aurmar_description/robots/ur16e.urdf (robot description, URDF)
Before this commit: robot ur, 12 links, 11 joints
Links:
- added link pod_base_link; visual mesh filename=package://Aurmar_description/meshes/pod/untitled.dae
Joints:
- added joint base_link-pod_base_link: type fixed, parent base_link, child pod_base_link, origin xyz=0.0 0 0 rpy=0 0 0

Commit message: Adding google scanned objects and each object with its varients

File: assets/urdf/Aurmar_description/robots/ur16e.urdf (robot description, URDF)
Before this commit: robot ur, 13 links, 12 joints
Links:
- link pod_base_link: geometry 

Commit message: Adding retract method for the target object

File: assets/urdf/Aurmar_description/robots/ur16e.urdf (robot description, URDF)
Before this commit: robot ur, 13 links, 12 joints
Links:
- link pod_base_link: geometry 
Joints:
- joint base_link-base_link_inertia: origin xyz=0 0 0 rpy=0 0 3.141592653589793 -> xyz=-0.05 0 0.05 rpy=0 0 3.141592653589793

Commit message: adding new retract mechanism for success and failure detection data collection

File: assets/urdf/Aurmar_description/robots/ur16e.urdf (robot description, URDF)
Before this commit: robot ur, 12 links, 11 joints
Links:
- added link pod_base_link
Joints:
- added joint base_link-pod_base_link: type fixed, parent base_link, child pod_base_link, origin xyz=0.0 0 0 rpy=0 0 0
- joint base_link-base_link_inertia: origin xyz=0 0 0 rpy=0 0 3.141592653589793 -> xyz=-0.05 0 0.05 rpy=0 0 3.141592653589793

Commit message: Lengthened eef rod

File: assets/urdf/Aurmar_description/robots/ur16e.urdf (robot description, URDF)
Before this commit: robot ur, 12 links, 11 joints
Links:
- link epick_rod: geometry collision cylinder length=0.13 radius=0.0065; visual cylinder length=0.13 radius=0.0065
Joints:
- joint eef_hand_joint: origin xyz=0 0 0.053 rpy=0 0 0 -> xyz=0 0 0.08 rpy=0 0 0

Commit message: Adding changes to the suction cup projection calucaltion and urdf file to shift the arm on left side by 5 cm

File: assets/urdf/Aurmar_description/robots/ur16e.urdf (robot description, URDF)
Before this commit: robot ur, 12 links, 11 joints
Joints:
- joint base_link-base_link_inertia: origin xyz=0 0 0 rpy=0 0 3.141592653589793 -> xyz=0 -0.05 0.05 rpy=0 0 3.141592653589793

Commit message: Adding new adjustments to the retract mechanism

File: assets/urdf/Aurmar_description/robots/ur16e.urdf (robot description, URDF)
Before this commit: robot ur, 13 links, 12 joints
Joints:
- joint base_link-base_link_inertia: origin xyz=-0.05 0 0.05 rpy=0 0 3.141592653589793 -> xyz=-0.05 -0.05 0.05 rpy=0 0 3.141592653589793
- joint eef_hand_joint: limit lower=0.0 upper=0.008 effort=1000.0 velocity=100 -> lower=0.0 upper=0.004 effort=1000.0 velocity=100

Commit message: Modifying the suction score calucaltor and adding different object list for different bins

File: assets/urdf/Aurmar_description/robots/ur16e.urdf (robot description, URDF)
Before this commit: robot ur, 13 links, 12 joints
Joints:
- joint eef_hand_joint: limit lower=0.0 upper=0.008 effort=1000.0 velocity=100 -> lower=0.0 upper=0.004 effort=1000.0 velocity=10000

Commit message: tweaks for better suction cup deformation score calucaltion and adding more checks for suction contact with the target object, adding continuous calcualtion of required force in every 10 sim step

File: assets/urdf/Aurmar_description/robots/ur16e.urdf (robot description, URDF)
Before this commit: robot ur, 13 links, 12 joints
Joints:
- joint eef_hand_joint: limit lower=0.0 upper=0.004 effort=1000.0 velocity=10000 -> lower=0.0 upper=0.0 effort=1000.0 velocity=1

Commit message: adding changes for better arm manipulability and changes for continuous suction score calculator

File: assets/urdf/Aurmar_description/robots/ur16e.urdf (robot description, URDF)
Before this commit: robot ur, 12 links, 11 joints
Links:
- added link pod_base_link
Joints:
- added joint base_link-pod_base_link: type fixed, parent base_link, child pod_base_link, origin xyz=0.0 0 0 rpy=0 0 0
- joint base_link-base_link_inertia: origin xyz=0 -0.05 0.05 rpy=0 0 3.141592653589793 -> xyz=-0.05 -0.05 0.05 rpy=0 0 3.141592653589793
- joint eef_hand_joint: limit lower=0.0 upper=0.008 effort=1000.0 velocity=100 -> lower=0.0 upper=0.0 effort=1000.0 velocity=1

Commit message: Changes: 1. Adding the vit training model 2. Editing the ur16e urdf file as it contained ur10e meshes 3. Fixing few syntax error related to data path 4. Changed the gitignore file and setup.py file

File: assets/urdf/Aurmar_description/robots/ur16e.urdf (robot description, URDF)
Before this commit: robot ur, 13 links, 12 joints
Links:
- link base_link_inertia: geometry collision mesh filename=package://Aurmar_description/meshes/ur16e/collision/base.stl; visual mesh filename=package://Aurmar_description/meshes/ur16e/visual/base.dae
- link shoulder_link: geometry collision mesh filename=meshes/ur16e/collision/shoulder.stl; visual mesh filename=meshes/ur16e/visual/shoulder.dae
- link wrist_1_link: geometry collision mesh filename=meshes/ur16e/collision/wrist1.stl; visual mesh filename=meshes/ur16e/visual/wrist1.dae
- link wrist_2_link: geometry collision mesh filename=meshes/ur16e/collision/wrist2.stl; visual mesh filename=meshes/ur16e/visual/wrist2.dae
- link wrist_3_link: geometry collision mesh filename=meshes/ur16e/collision/wrist3.stl; visual mesh filename=meshes/ur16e/visual/wrist3.dae
