Commit message: Complete reset when timed out + larger objects

File: assets/urdf_models/models/centrum_box_1/model.urdf (robot description, URDF)
Before this commit: robot model.urdf, 1 links, 0 joints
Links:
- link baseLink: geometry collision box size=0.11 0.065 0.065; visual box size=0.11 0.065 0.065

File: assets/urdf_models/models/centrum_box_2/model.urdf (robot description, URDF)
Before this commit: robot model.urdf, 1 links, 0 joints
Links:
- link baseLink: geometry collision box size=0.11 0.065 0.065; visual box size=0.11 0.065 0.065

File: assets/urdf_models/models/centrum_box_3/model.urdf (robot description, URDF)
Before this commit: robot model.urdf, 1 links, 0 joints
Links:
- link baseLink: geometry collision box size=0.11 0.065 0.065; visual box size=0.11 0.065 0.065

File: assets/urdf_models/models/centrum_box_4/model.urdf (robot description, URDF)
Before this commit: robot model.urdf, 1 links, 0 joints
Links:
- link baseLink: geometry collision box size=0.11 0.065 0.065; visual box size=0.11 0.065 0.065

File: assets/urdf_models/models/centrum_box_5/model.urdf (robot description, URDF)
Before this commit: robot model.urdf, 1 links, 0 joints
Links:
- link baseLink: geometry collision box size=0.11 0.065 0.065; visual box size=0.11 0.065 0.065

File: assets/urdf_models/models/kyolic_bottle_1/model.urdf (robot description, URDF)
Before this commit: robot model.urdf, 1 links, 0 joints
Links:
- link baseLink: geometry collision cylinder length=0.107 radius=0.045; visual cylinder length=0.107 radius=0.045

File: assets/urdf_models/models/kyolic_bottle_2/model.urdf (robot description, URDF)
Before this commit: robot model.urdf, 1 links, 0 joints
Links:
- link baseLink: geometry collision cylinder length=0.107 radius=0.045; visual cylinder length=0.107 radius=0.045

File: assets/urdf_models/models/kyolic_bottle_3/model.urdf (robot description, URDF)
Before this commit: robot model.urdf, 1 links, 0 joints
Links:
- link baseLink: geometry collision cylinder length=0.107 radius=0.045; visual cylinder length=0.107 radius=0.045

File: assets/urdf_models/models/kyolic_bottle_4/model.urdf (robot description, URDF)
Before this commit: robot model.urdf, 1 links, 0 joints
Links:
- link baseLink: geometry collision cylinder length=0.107 radius=0.045; visual cylinder length=0.107 radius=0.045

File: assets/urdf_models/models/kyolic_bottle_5/model.urdf (robot description, URDF)
Before this commit: robot model.urdf, 1 links, 0 joints
Links:
- link baseLink: geometry collision cylinder length=0.107 radius=0.045; visual cylinder length=0.107 radius=0.045

File: assets/urdf_models/models/realsense_box_1/model.urdf (robot description, URDF)
Before this commit: robot model.urdf, 1 links, 0 joints
Links:
- link baseLink: geometry collision box size=0.165 0.096 0.072; visual box size=0.165 0.096 0.072

File: assets/urdf_models/models/realsense_box_2/model.urdf (robot description, URDF)
Before this commit: robot model.urdf, 1 links, 0 joints
Links:
- link baseLink: geometry collision box size=0.165 0.096 0.072; visual box size=0.165 0.096 0.072

File: assets/urdf_models/models/realsense_box_3/model.urdf (robot description, URDF)
Before this commit: robot model.urdf, 1 links, 0 joints
Links:
- link baseLink: geometry collision box size=0.165 0.096 0.072; visual box size=0.165 0.096 0.072

File: assets/urdf_models/models/realsense_box_4/model.urdf (robot description, URDF)
Before this commit: robot model.urdf, 1 links, 0 joints
Links:
- link baseLink: geometry collision box size=0.165 0.096 0.072; visual box size=0.165 0.096 0.072

File: assets/urdf_models/models/realsense_box_5/model.urdf (robot description, URDF)
Before this commit: robot model.urdf, 1 links, 0 joints
Links:
- link baseLink: geometry collision box size=0.165 0.096 0.072; visual box size=0.165 0.096 0.072

File: assets/urdf_models/models/small_health_bottle_1/model.urdf (robot description, URDF)
Before this commit: robot model.urdf, 1 links, 0 joints
Links:
- link baseLink: geometry collision cylinder length=0.099 radius=0.045; visual cylinder length=0.099 radius=0.045

File: assets/urdf_models/models/small_health_bottle_2/model.urdf (robot description, URDF)
Before this commit: robot model.urdf, 1 links, 0 joints
Links:
- link baseLink: geometry collision cylinder length=0.099 radius=0.045; visual cylinder length=0.099 radius=0.045

File: assets/urdf_models/models/small_health_bottle_3/model.urdf (robot description, URDF)
Before this commit: robot model.urdf, 1 links, 0 joints
Links:
- link baseLink: geometry collision cylinder length=0.099 radius=0.045; visual cylinder length=0.099 radius=0.045

File: assets/urdf_models/models/small_health_bottle_4/model.urdf (robot description, URDF)
Before this commit: robot model.urdf, 1 links, 0 joints
Links:
- link baseLink: geometry collision cylinder length=0.099 radius=0.045; visual cylinder length=0.099 radius=0.045

File: assets/urdf_models/models/small_health_bottle_5/model.urdf (robot description, URDF)
Before this commit: robot model.urdf, 1 links, 0 joints
Links:
- link baseLink: geometry collision cylinder length=0.099 radius=0.045; visual cylinder length=0.099 radius=0.045
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