Commit message: Reset suction flag + new test obj list

File: assets/urdf_models/models/realsense_box_1/model.urdf (robot description, URDF)
Before this commit: robot model.urdf, 1 links, 0 joints
Links:
- link baseLink: geometry collision box size=0.165 0.096 0.085; visual box size=0.165 0.096 0.085

File: assets/urdf_models/models/realsense_box_2/model.urdf (robot description, URDF)
Before this commit: robot model.urdf, 1 links, 0 joints
Links:
- link baseLink: geometry collision box size=0.165 0.096 0.085; visual box size=0.165 0.096 0.085

File: assets/urdf_models/models/realsense_box_3/model.urdf (robot description, URDF)
Before this commit: robot model.urdf, 1 links, 0 joints
Links:
- link baseLink: geometry collision box size=0.165 0.096 0.085; visual box size=0.165 0.096 0.085

File: assets/urdf_models/models/realsense_box_4/model.urdf (robot description, URDF)
Before this commit: robot model.urdf, 1 links, 0 joints
Links:
- link baseLink: geometry collision box size=0.165 0.096 0.085; visual box size=0.165 0.096 0.085

File: assets/urdf_models/models/realsense_box_5/model.urdf (robot description, URDF)
Before this commit: robot model.urdf, 1 links, 0 joints
Links:
- link baseLink: geometry collision box size=0.165 0.096 0.085; visual box size=0.165 0.096 0.085
