Commit message: Removed false negatives from spawning objects

File: assets/urdf_models/models/pizza_cutter_1/model.urdf (robot description, URDF)
Before this commit: robot model.urdf, 1 links, 0 joints
Links:
- link baseLink: geometry collision box size=0.135 0.105 0.085; visual box size=0.135 0.105 0.085

File: assets/urdf_models/models/pizza_cutter_2/model.urdf (robot description, URDF)
Before this commit: robot model.urdf, 1 links, 0 joints
Links:
- link baseLink: geometry collision box size=0.135 0.105 0.085; visual box size=0.135 0.105 0.085

File: assets/urdf_models/models/pizza_cutter_3/model.urdf (robot description, URDF)
Before this commit: robot model.urdf, 1 links, 0 joints
Links:
- link baseLink: geometry collision box size=0.135 0.105 0.085; visual box size=0.135 0.105 0.085

File: assets/urdf_models/models/pizza_cutter_4/model.urdf (robot description, URDF)
Before this commit: robot model.urdf, 1 links, 0 joints
Links:
- link baseLink: geometry collision box size=0.135 0.105 0.085; visual box size=0.135 0.105 0.085

File: assets/urdf_models/models/pizza_cutter_5/model.urdf (robot description, URDF)
Before this commit: robot model.urdf, 1 links, 0 joints
Links:
- link baseLink: geometry collision box size=0.135 0.105 0.085; visual box size=0.135 0.105 0.085
