Commit message: multi obj

File: assets/urdf_models/models/small_health_bottle_1/model.urdf (robot description, URDF)
Before this commit: robot model.urdf, 1 links, 0 joints
Links:
- link baseLink: geometry collision cylinder length=0.099 radius=0.055; visual cylinder length=0.099 radius=0.055

File: assets/urdf_models/models/small_health_bottle_2/model.urdf (robot description, URDF)
Before this commit: robot model.urdf, 1 links, 0 joints
Links:
- link baseLink: geometry collision cylinder length=0.099 radius=0.055; visual cylinder length=0.099 radius=0.055

File: assets/urdf_models/models/small_health_bottle_3/model.urdf (robot description, URDF)
Before this commit: robot model.urdf, 1 links, 0 joints
Links:
- link baseLink: geometry collision cylinder length=0.099 radius=0.055; visual cylinder length=0.099 radius=0.055

File: assets/urdf_models/models/small_health_bottle_4/model.urdf (robot description, URDF)
Before this commit: robot model.urdf, 1 links, 0 joints
Links:
- link baseLink: geometry collision cylinder length=0.099 radius=0.055; visual cylinder length=0.099 radius=0.055

File: assets/urdf_models/models/small_health_bottle_5/model.urdf (robot description, URDF)
Before this commit: robot model.urdf, 1 links, 0 joints
Links:
- link baseLink: geometry collision cylinder length=0.099 radius=0.055; visual cylinder length=0.099 radius=0.055

Commit message: fixed: fixed scnene

File: assets/urdf_models/models/small_health_bottle_1/model.urdf (robot description, URDF)
Before this commit: robot model.urdf, 1 links, 0 joints
Links:
- link baseLink: geometry collision cylinder length=0.099 radius=0.065; visual cylinder length=0.099 radius=0.065

File: assets/urdf_models/models/small_health_bottle_2/model.urdf (robot description, URDF)
Before this commit: robot model.urdf, 1 links, 0 joints
Links:
- link baseLink: mass 0.113 -> 0.108; geometry collision cylinder length=0.099 radius=0.065; visual cylinder length=0.099 radius=0.065

File: assets/urdf_models/models/small_health_bottle_3/model.urdf (robot description, URDF)
Before this commit: robot model.urdf, 1 links, 0 joints
Links:
- link baseLink: mass 0.118 -> 0.108; geometry collision cylinder length=0.099 radius=0.065; visual cylinder length=0.099 radius=0.065

File: assets/urdf_models/models/small_health_bottle_4/model.urdf (robot description, URDF)
Before this commit: robot model.urdf, 1 links, 0 joints
Links:
- link baseLink: mass 0.123 -> 0.108; geometry collision cylinder length=0.099 radius=0.065; visual cylinder length=0.099 radius=0.065

File: assets/urdf_models/models/small_health_bottle_5/model.urdf (robot description, URDF)
Before this commit: robot model.urdf, 1 links, 0 joints
Links:
- link baseLink: mass 0.128 -> 0.108; geometry collision cylinder length=0.099 radius=0.065; visual cylinder length=0.099 radius=0.065
