Commit message: Diverse obj scenes

File: assets/urdf_models/models/blue_cup_1/model.urdf (robot description, URDF)
Before this commit: robot model.urdf, 1 links, 0 joints
Links:
- link baseLink: geometry collision mesh filename=collision.obj scale=1.2 1.2 1.2; visual mesh filename=textured.obj scale=1 1 1
