Commit message: Edited object size and target set to be graspable

File: assets/urdf_models/models/blue_tea_box_1/model.urdf (robot description, URDF)
Before this commit: robot model.urdf, 1 links, 0 joints
Links:
- link baseLink: geometry collision mesh filename=collision.obj scale=1.4 1.4 1.4; visual mesh filename=textured.obj scale=1.2 1.2 1.2
